Commit message: 初版（未实车测试）

File: rm_robot_description/urdf/rm_gimbal.urdf.xacro (robot description, xacro)
@@ -1,25 +1,62 @@
 <?xml version="1.0" encoding="utf-8"?>
-<robot name="rm_gimbal"
-  xmlns:xacro="http://ros.org/wiki/xacro">
-  <xacro:arg name="xyz" default="0.10 0 0.05" />
-  <xacro:arg name="rpy" default="0 0 0" />
+<robot name="rm_gimbal" xmlns:xacro="http://ros.org/wiki/xacro">
+  <!-- 相机0安装参数 -->
+  <xacro:arg name="camera0_xyz" default="0.10 0.0 0.05" />
+  <xacro:arg name="camera0_rpy" default="0.0 0.0 0.0" />
+  <!-- 后相机（相机1）安装参数：向后0.10m，高度与前相机一致 -->
+  <xacro:arg name="camera1_xyz" default="-0.10 0.0 0.05" />
+  <xacro:arg name="camera1_rpy" default="0.0 0.0 0.0" />
   <link name="odom" />
+  <!-- Yaw轴 -->
+  <link name="yaw_link" />
+  <joint name="yaw_joint" type="revolute">
+    <parent link="odom" />
+    <child link="yaw_link" />
+    <origin xyz="0 0 0" rpy="0 0 0" />
+    <axis xyz="0 0 1" />
+    <limit lower="-3.14" upper="3.14" effort="100" velocity="10" />
+  </joint>
+  <!-- Pitch轴 -->
+  <link name="pitch_link" />
+  <joint name="pitch_joint" type="revolute">
+    <parent link="yaw_link" />
+    <child link="pitch_link" />
+    <origin xyz="0 0 0" rpy="0 0 0" />
+    <axis xyz="0 1 0" />
+    <limit lower="-1.57" upper="1.57" effort="100" velocity="10" />
+  </joint>
+  <!-- 兼容层 gimbal_link -->
   <link name="gimbal_link" />
-  <joint name="gimbal_joint" type="floating">
-    <parent link="odom" />
+  <joint name="gimbal_joint" type="fixed">
+    <parent link="pitch_link" />
     <child link="gimbal_link" />
+    <origin xyz="0 0 0" rpy="0 0 0" />
   </joint>
-  <link name="camera_link" />
-  <joint name="camera_joint" type="fixed">
-    <origin xyz="$(arg xyz)" rpy="$(arg rpy)" />
+  <!-- 前相机（相机0） -->
+  <link name="camera_0_link" />
+  <joint name="camera_0_joint" type="fixed">
+    <origin xyz="$(arg camera0_xyz)" rpy="$(arg camera0_rpy)" />
     <parent link="gimbal_link" />
-    <child link="camera_link" />
-    <axis xyz="0 0 0" />
+    <child link="camera_0_link" />
   </joint>
-  <link name="camera_optical_frame" />
-  <joint name="camera_optical_joint" type="fixed">
+  <link name="camera_0_optical_frame" />
+  <joint name="camera_0_optical_joint" type="fixed">
     <origin xyz="0 0 0" rpy="${-pi/2} 0 ${-pi/2}" />
-    <parent link="camera_link" />
-    <child link="camera_optical_frame" />
+    <parent link="camera_0_link" />
+    <child link="camera_0_optical_frame" />
+  </joint>
+  <!-- 后相机（相机1） -->
+  <link name="camera_1_link" />
+  <joint name="camera_1_joint" type="fixed">
+    <origin xyz="$(arg camera1_xyz)" rpy="$(arg camera1_rpy)" />
+    <parent link="gimbal_link" />
+    <child link="camera_1_link" />
+  </joint>
+  <link name="camera_1_optical_frame" />
+  <joint name="camera_1_optical_joint" type="fixed">
+    <!-- 注意：后相机光轴向后，需绕Y轴额外转180°，即 RPY = (-pi/2, 0, pi/2) -->
+    <origin xyz="0 0 0" rpy="${-pi/2} 0 ${pi/2}" />
+    <parent link="camera_1_link" />
+    <child link="camera_1_optical_frame" />
   </joint>
 </robot>
